Commit message: Check point commit

File: data/urdf/DARwInOP.urdf (robot description, URDF)
Before this commit: robot darwinOP, 25 links, 24 joints
Joints:
- joint j_ankle1_l: limit lower=-2.6179939 upper=2.6179939 effort=10 velocity=5.6548668 -> lower=-2.6179939 upper=2.6179939 effort=2.8 velocity=5.6548668
- joint j_ankle1_r: limit lower=-2.6179939 upper=2.6179939 effort=10 velocity=5.6548668 -> lower=-2.6179939 upper=2.6179939 effort=2.8 velocity=5.6548668
- joint j_ankle2_l: limit lower=-2.6179939 upper=2.6179939 effort=10 velocity=5.6548668 -> lower=-2.6179939 upper=2.6179939 effort=2.8 velocity=5.6548668
- joint j_ankle2_r: limit lower=-2.6179939 upper=2.6179939 effort=10 velocity=5.6548668 -> lower=-2.6179939 upper=2.6179939 effort=2.8 velocity=5.6548668
- joint j_pelvis_l: limit lower=-2.6179939 upper=2.6179939 effort=10 velocity=5.6548668 -> lower=-2.6179939 upper=2.6179939 effort=2.8 velocity=5.6548668
- joint j_pelvis_r: limit lower=-2.6179939 upper=2.6179939 effort=10 velocity=5.6548668 -> lower=-2.6179939 upper=2.6179939 effort=2.8 velocity=5.6548668
- joint j_thigh1_l: limit lower=-2.6179939 upper=2.6179939 effort=10 velocity=5.6548668 -> lower=-2.6179939 upper=2.6179939 effort=2.8 velocity=5.6548668
- joint j_thigh1_r: limit lower=-2.6179939 upper=2.6179939 effort=10 velocity=5.6548668 -> lower=-2.6179939 upper=2.6179939 effort=2.8 velocity=5.6548668
- joint j_thigh2_l: limit lower=-2.6179939 upper=2.6179939 effort=10 velocity=5.6548668 -> lower=-2.6179939 upper=2.6179939 effort=2.8 velocity=5.6548668
- joint j_thigh2_r: limit lower=-2.6179939 upper=2.6179939 effort=10 velocity=5.6548668 -> lower=-2.6179939 upper=2.6179939 effort=2.8 velocity=5.6548668
- joint j_tibia_l: limit lower=-2.6179939 upper=2.6179939 effort=10 velocity=5.6548668 -> lower=-2.6179939 upper=0.0009939 effort=2.8 velocity=5.6548668
- joint j_tibia_r: limit lower=-2.6179939 upper=2.6179939 effort=10 velocity=5.6548668 -> lower=-0.0009939 upper=2.6179939 effort=2.8 velocity=5.6548668

Commit message: Fixed joint limit

File: data/urdf/DARwInOP.urdf (robot description, URDF)
Before this commit: robot darwinOP, 25 links, 24 joints
Joints:
- joint j_ankle1_l: limit lower=-2.6179939 upper=2.6179939 effort=2.8 velocity=5.6548668 -> lower=-1.5 upper=0.7 effort=2.8 velocity=5.6548668
- joint j_ankle1_r: limit lower=-2.6179939 upper=2.6179939 effort=2.8 velocity=5.6548668 -> lower=-0.7 upper=1.5 effort=2.8 velocity=5.6548668
- joint j_ankle2_l: limit lower=-2.6179939 upper=2.6179939 effort=2.8 velocity=5.6548668 -> lower=-0.7 upper=0.7 effort=2.8 velocity=5.6548668
- joint j_ankle2_r: limit lower=-2.6179939 upper=2.6179939 effort=2.8 velocity=5.6548668 -> lower=-0.7 upper=0.7 effort=2.8 velocity=5.6548668
- joint j_back_l: limit lower=-2.6179939 upper=2.6179939 effort=2.8 velocity=5.6548668 -> (none)
- joint j_back_r: limit lower=-2.6179939 upper=2.6179939 effort=2.8 velocity=5.6548668 -> (none)
- joint j_camboard: limit lower=-2.6179939 upper=2.6179939 effort=2.8 velocity=5.6548668 -> (none)
- joint j_high_arm_l: limit lower=-2.6179939 upper=2.6179939 effort=2.8 velocity=5.648668 -> lower=-1.5707963 upper=1.5707963 effort=2.8 velocity=5.648668
- joint j_high_arm_r: limit lower=-2.6179939 upper=2.6179939 effort=2.8 velocity=5.648668 -> lower=-1.5707963 upper=1.5707963 effort=2.8 velocity=5.648668
- joint j_low_arm_l: limit lower=-2.6179939 upper=2.6179939 effort=2.8 velocity=5.6548668 -> lower=-2.6179939 upper=0 effort=2.8 velocity=5.6548668
- joint j_low_arm_r: limit lower=-1.635 upper=2.6179939 effort=2.8 velocity=5.6548668 -> lower=0 upper=2.6179939 effort=2.8 velocity=5.6548668
- joint j_pan: limit lower=-2.6179939 upper=2.6179939 effort=2.8 velocity=5.6548668 -> lower=-1.5707963 upper=1.5707963 effort=2.8 velocity=5.6548668
- joint j_pelvis_l: limit lower=-2.6179939 upper=2.6179939 effort=2.8 velocity=5.6548668 -> lower=-0.7853981 upper=0.7853981 effort=2.8 velocity=5.6548668
- joint j_pelvis_r: limit lower=-2.6179939 upper=2.6179939 effort=2.8 velocity=5.6548668 -> lower=-0.7853981 upper=0.7853981 effort=2.8 velocity=5.6548668
- joint j_thigh1_l: limit lower=-2.6179939 upper=2.6179939 effort=2.8 velocity=5.6548668 -> lower=-1.5707963 upper=1.5707963 effort=2.8 velocity=5.6548668
- joint j_thigh1_r: limit lower=-2.6179939 upper=2.6179939 effort=2.8 velocity=5.6548668 -> lower=-1.5707963 upper=1.5707963 effort=2.8 velocity=5.6548668
- joint j_thigh2_l: limit lower=-2.6179939 upper=2.6179939 effort=2.8 velocity=5.6548668 -> lower=-0.3926991 upper=1.5707963 effort=2.8 velocity=5.6548668
- joint j_thigh2_r: limit lower=-2.6179939 upper=2.6179939 effort=2.8 velocity=5.6548668 -> lower=-1.5707963 upper=0.3926991 effort=2.8 velocity=5.6548668
- joint j_tibia_l: limit lower=-2.6179939 upper=0.0009939 effort=2.8 velocity=5.6548668 -> lower=-2.6548668 upper=0 effort=2.8 velocity=5.6548668
- joint j_tibia_r: limit lower=-0.0009939 upper=2.6179939 effort=2.8 velocity=5.6548668 -> lower=0 upper=2.6179939 effort=2.8 velocity=5.6548668
- joint j_tilt: limit lower=-2.6179939 upper=2.6179939 effort=2.8 velocity=5.6548668 -> lower=-0.3926991 upper=0.7853981 effort=2.8 velocity=5.6548668
